Commit message: Add README documentation and project files

File: install/ur_description/share/ur_description/urdf/ur_macro.xacro (robot description, xacro)
@@ -14,5 +14,6 @@
     safety_pos_margin:=0.15
     safety_k_position:=20
-    force_abs_paths:=false
+    force_abs_paths:=false,
+    skip_base_joint:=false
     ">
     <!-- Load configuration data from the provided .yaml files -->
@@ -207,9 +208,11 @@
     </link>
     <!-- base_joint fixes base_link to the environment -->
-    <joint name="${tf_prefix}base_joint" type="fixed">
-      <xacro:insert_block name="origin" />
-      <parent link="${parent}" />
-      <child link="${tf_prefix}base_link" />
-    </joint>
+    <xacro:unless value="${skip_base_joint}">
+      <joint name="${tf_prefix}base_joint" type="fixed">
+        <xacro:insert_block name="origin" />
+        <parent link="${parent}" />
+        <child link="${tf_prefix}base_link" />
+      </joint>
+    </xacro:unless>
     <!-- joints - main serial chain -->
     <joint name="${tf_prefix}base_link-base_link_inertia" type="fixed">

File: install/ur_description/share/ur_description/urdf/ur_robotiq_140.urdf.xacro (robot description, xacro)
@@ -36,5 +36,5 @@
      safety_k_position="$(arg safety_k_position)"
      force_abs_paths="$(arg force_abs_paths)">
-     <origin xyz="0 0 0" rpy="0 0 0" /> <!-- Position robot in the world (Handled by Spawn args) -->
+     <origin xyz="0 0.2 0.8" rpy="0 0 0" /> <!-- Position robot in the world -->
    </xacro:ur_robot>
    <!-- Instantiate Robotiq 140 Gripper -->

File: src/ur_description/urdf/ur_robotiq_140.urdf.xacro (robot description, xacro)
@@ -22,13 +22,19 @@
    <xacro:include filename="$(find robotiq_2f_gripper_description)/urdf/robotiq_2f_140_macro.xacro" />
    <!-- Create link fixed to the "world" -->
-   <!-- <link name="world" /> -->
+   <link name="world" />
    <!-- Arm -->
    <xacro:ur_robot
      name="$(arg name)"
      tf_prefix="$(arg tf_prefix)"
+     parent="world"
+     joint_limits_parameters_file="$(arg joint_limit_params)"
+     kinematics_parameters_file="$(arg kinematics_params)"
+     physical_parameters_file="$(arg physical_params)"
+     visual_parameters_file="$(arg visual_params)"
+     safety_limits="$(arg safety_limits)"
+     safety_pos_margin="$(arg safety_pos_margin)"
      safety_k_position="$(arg safety_k_position)"
-     force_abs_paths="$(arg force_abs_paths)"
-     skip_base_joint="true">
-     <origin xyz="0 0 0" rpy="0 0 0" /> <!-- Ignored when skip_base_joint is true -->
+     force_abs_paths="$(arg force_abs_paths)">
+     <origin xyz="0 0.2 0.8" rpy="0 0 0" /> <!-- Position robot in the world -->
    </xacro:ur_robot>
    <!-- Instantiate Robotiq 140 Gripper -->
