Commit message: Remove visual from shoulder_link in ur.urdf
Removed visual element from shoulder_link in URDF.

File: src/ur_description/urdf/ur.urdf (robot description, URDF)
Before this commit: robot ur_robotiq_140, 24 links, 23 joints
Links:
- link shoulder_link: geometry collision mesh filename=package://ur_description/meshes/ur3e/collision/shoulder.stl
